File: hardware/ch32v003f4u6_with_wsled/ch32v003f4u6_with_wsled.kicad_pcb (KiCad board)
At the start: 2 copper layers, 30.5 x 43.2 mm, 24 parts, among them J2 PGM, J4 USB_C_Receptacle_USB2.0, J5 HOLE, M1 Mic, U1 CH32V003F4U6, U2 3.3vReg

Commit message: Update routed hardware design
Parts:
- added C5: 1u, Capacitor_SMD:C_0402_1005Metric, F.Cu at (95.0, 91.0)
- added J6: HOLE, MountingHole:MountingHole_2.2mm_M2_DIN965_Pad, F.Cu at (92.5, 109.0)
- added R7: 0, Resistor_SMD:R_0402_1005Metric, F.Cu at (96.2, 92.7)
- added R8: 0, Resistor_SMD:R_0402_1005Metric, F.Cu at (93.0, 92.0)
- moved C3 7.96 mm to (97.5, 94.9), turned to 30 degrees
- moved R5 7.85 mm to (102.1, 94.5), turned to 180 degrees
- moved C4 2.34 mm to (103.5, 86.8), turned to 160 degrees
- moved C1 1.88 mm to (96.6, 100.5)
- moved R6 1.71 mm to (94.3, 93.0), turned to -175 degrees
- moved J2 1.27 mm to (94.9, 114.0)
- moved U2 0.74 mm to (103.0, 88.5)
- moved J5 0.72 mm to (107.5, 89.0)
- moved M1 0.67 mm to (92.5, 89.0)
- turned U1 to -47 degrees
Connections:
- D1 pad 3: +5V -> VCC
- D2 pad 3: +5V -> VCC
- D3 pad 3: +5V -> VCC
- D4 pad 3: +5V -> VCC
- D5 pad 3: +5V -> VCC
- D6 pad 3: +5V -> VCC
- J2 pad 3: PD7NRST -> VCC
- M1 pad 2: PA1 -> Net-(M1-Pad2)
- R6 pad 1: VCC -> Net-(R6-Pad1)
- R6 pad 2: PA1 -> Net-(M1-Pad2)
Routing:
- net GND: track 0.00 -> 159.8 mm, vias 0 -> 84
- net VCC: track 0.00 -> 68.5 mm, vias 0 -> 11
- net +5V: track 0.00 -> 67.5 mm, vias 0 -> 2
- net SWIO: track 0.00 -> 29.5 mm, vias 0 -> 2
- net PC6: track 0.00 -> 28.5 mm, vias 0 -> 2
- net D-: track 0.00 -> 23.6 mm, vias 0 -> 2
- net PA1: track 0.00 -> 21.1 mm
- net DPU: track 0.00 -> 18.8 mm, vias 0 -> 2
- net PD7NRST: track 0.00 -> 17.5 mm, vias 0 -> 1
- net D+: track 0.00 -> 17.3 mm
- net PD6: track 0.00 -> 17.1 mm, vias 0 -> 2
- net Net-(J4-PadA6): track 0.00 -> 16.5 mm, vias 0 -> 2
- net PC4: track 0.00 -> 16.2 mm, vias 0 -> 1
- net PC5: track 0.00 -> 15.4 mm, vias 0 -> 1
- net PC3: track 0.00 -> 15.1 mm, vias 0 -> 2
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- added copper zone on B.Cu, net GND
- added copper zone on F.Cu, net GND
Other:
- board size 30.5 x 43.2 mm -> 35.6 x 44.5 mm
- board text added: "003f4u6"
- board text added: "CPU"
- board text added: "GND SWIO 3.3v 5V GND"
- board text added: "Microphone"
- board text added: "NRST PA1 PA2 GND PD0 VCC PC0 PC1 PC2 PC3"
- board text added: "PD6 PD5 PD4 PD3 P2 SWIO PC7 PC6 PC5 PC4"
- board text added: "These 6 are LEDs"
- board text added: "ch32v003_fun"
