File: hardware/ch32v003f4u6_with_wsled/ch32v003f4u6_with_wsled.kicad_sch (KiCad schematic)
At the start: 24 parts, among them J2 PGM, J4 USB_C_Receptacle_USB2.0, J5 HOLE, M1 Mic, U1 CH32V003F4U6, U2 3.3vReg

Commit message: Update routed hardware design
Parts:
- added C5: 1u, Capacitor_SMD:C_0402_1005Metric, symbol Device:C
- added J6: HOLE, MountingHole:MountingHole_2.2mm_M2_DIN965_Pad, symbol Connector_Generic:Conn_01x01
- added R7, R8: 0, Resistor_SMD:R_0402_1005Metric, symbol Device:R
Connections:
- net +5V: no longer D1.3 (V), D2.3 (V), D3.3 (V), D4.3 (V), D5.3 (V), D6.3 (V)
- net GND: now also C5.1, J6.1 (Pin_1)
- net PA1: now also R8.1; no longer M1.2 (Pin_2), R6.2
- net PD7NRST: no longer J2.3 (Pin_3)
- net VCC: now also D1.3 (V), D2.3 (V), D3.3 (V), D4.3 (V), D5.3 (V), D6.3 (V), J2.3 (Pin_3), R7.1; no longer R6.1
- new net: M1.2 (Pin_2), R6.2, R8.2
- new net: C5.2, R6.1, R7.2
