File: hardware/ch32v003f4u6_pendant/ch32v003f4u6_pendant.kicad_pcb (KiCad board)
At the start: 2 copper layers, 20.3 x 51.4 mm, 54 parts, among them J1 USB_C_Receptacle_USB2.0, J2 BONUS, J3 BONUS, J4 CONN, J7 BATT, J9 GND, Q1 Q_Photo_NPN, Q2 NMOS, T1 TOUCHPAD, U1 MD5112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

Commit message: Update pendant
Parts:
- removed J9: GND, TestPoint:TestPoint_Loop_D1.80mm_Drill1.0mm_Beaded
- removed MIC1: Mic, Swadge_Parts:GOERTEK_MIC_B4013AM423
- removed R7: 2.2k, Resistor_SMD:R_0201_0603Metric
- added U7: S08OB383-031, GOERTEK-S08OB383-031-MemsMic:GOERTEK-S08OB383-031-MemsMic, F.Cu at (91.4, 67.4)
- J4: moved to B.Cu
- moved C16 22.9 mm to (104.6, 31.3), turned to -90 degrees
- moved R16 18.2 mm to (94.3, 62.8), turned to 0 degrees
- moved C2 4.10 mm to (91.3, 63.9), turned to 180 degrees
- moved C14 2.91 mm to (95.3, 55.2), turned to 90 degrees
- moved U6 2.89 mm to (96.9, 55.2), turned to 180 degrees
- moved C11 2.79 mm to (96.9, 53.7), turned to 180 degrees
- moved R9 1.86 mm to (95.0, 48.0)
- moved R11 1.63 mm to (89.9, 32.8)
- moved C6 1.25 mm to (103.3, 56.9)
- moved R13 1.04 mm to (99.6, 55.8)
- moved T1 1.03 mm to (98.7, 72.8)
- moved R3 1.02 mm to (103.3, 49.6)
- moved R5 1.02 mm to (102.1, 49.5)
- moved C7 1.02 mm to (97.0, 59.4)
- moved R12 1.02 mm to (102.1, 55.4)
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Connections:
- D1 pad 1: unconnected-(D1-Pad1) -> GND
- D1 pad 5: unconnected-(D1-Pad5) -> Net-(D1-Pad5)
- D2 pad 1: unconnected-(D2-Pad1) -> Net-(D1-Pad5)
Routing:
- net GND: track 0.00 -> 147.5 mm, vias 0 -> 74
- net VD: track 0.00 -> 71.3 mm, vias 0 -> 6
- net VDD: track 0.00 -> 60.3 mm, vias 0 -> 5
- net PHOTODIODE: track 0.00 -> 42.6 mm, vias 0 -> 5
- net WSOUT: track 0.00 -> 39.5 mm, vias 0 -> 1
- net TOUCH: track 0.00 -> 38.9 mm, vias 0 -> 1
- net VCC: track 0.00 -> 38.7 mm, vias 0 -> 2
- net BONUS1: track 0.00 -> 29.1 mm
- net BONUS2: track 0.00 -> 25.8 mm, vias 0 -> 1
- net Net-(J1-PadA6): track 0.00 -> 22.5 mm, vias 0 -> 2
- net SCL: track 0.00 -> 20.6 mm, vias 0 -> 2
- net VCCMON: track 0.00 -> 19.9 mm, vias 0 -> 2
- net PD6: track 0.00 -> 19.7 mm, vias 0 -> 2
- net PD2: track 0.00 -> 19.6 mm, vias 0 -> 1
- net Net-(J1-PadA7): track 0.00 -> 18.4 mm, vias 0 -> 2
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- added copper zone on B.Cu, net GND
- added copper zone on F.Cu, net GND

Commit message: Update hardware
Parts:
- L1, L2: value 10uH -> 4.7uH
- moved R17 0.11 mm to (94.9, 50.9)
Routing:
- net GND: track 147.5 -> 156.3 mm, vias 74 -> 78
- net PHOTODIODE: track 42.6 -> 40.7 mm
- net VCC: track 38.7 -> 37.5 mm
- net VD: track 71.3 -> 70.5 mm
- net VDD: track 60.3 -> 59.6 mm
- net Net-(C1-Pad1): track 12.1 -> 11.4 mm
- net TOUCH: track 38.9 -> 38.3 mm
- net NRST: track 12.5 -> 13.0 mm
Other:
- board text added: "ch32v003fun ch32v003f4u6_pendant rev -"

Commit message: Update design a little
Parts:
- Q2: footprint Package_TO_SOT_SMD:SOT-323_SC-70 -> DFN-3L-1x0.6:DFN-3L-1x0.6
- moved Q2 0.70 mm to (100.0, 44.8), turned to -90 degrees
Routing:
- net T2CH4: track 3.84 -> 5.15 mm
- net GND: track 156.3 -> 156.9 mm
