File: hardware/ch32v003f4u6_pendant/ch32v003f4u6_pendant.kicad_sch (KiCad schematic)
At the start: 54 parts, among them J1 USB_C_Receptacle_USB2.0, J2 BONUS, J3 BONUS, J4 CONN, J7 BATT, J9 GND, Q1 Q_Photo_NPN, Q2 NMOS, T1 TOUCHPAD, U1 MD5112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

Commit message: Update pendant
Parts:
- removed J9: GND, TestPoint:TestPoint_Loop_D1.80mm_Drill1.0mm_Beaded, symbol Connector_Generic:Conn_01x01
- removed MIC1: Mic, Swadge_Parts:GOERTEK_MIC_B4013AM423, symbol Connector_Generic:Conn_01x02
- removed R7: 2.2k, Resistor_SMD:R_0201_0603Metric, symbol Device:R
- added U7: S08OB383-031, GOERTEK-S08OB383-031-MemsMic:GOERTEK-S08OB383-031-MemsMic, symbol GOERTEK-S08OB383-031-MemsMic:S08OB383-031
- Q1: LCSC (none) -> C100090
Connections:
- net GND: now also D1.1 (BI), U7.2 (GND), U7.3 (GND), U7.5 (GND), U7.6 (GND)
- net PD6: now also U7.4 (PWR)
- net at D1.5 (BO): now also D2.1 (BI)
- net at C2.2: now also U7.1 (OUT)
Other:
- note added: "TODO: Swap Microphone? C233789"
- moved on the sheet: C2

Commit message: Update hardware
Parts:
- L1, L2: value 10uH -> 4.7uH; LCSC C356837 -> C379996
Other:
- note removed: "TODO: Swap Microphone? C233789"
Changed lines of the file:
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@@
     (effects (font (size 2.54 2.54) (thickness 0.508) bold) (justify left bottom))
-  )
-  (text "TODO: Swap Microphone?\nC233789" (at 308.61 90.17 0)
-    (effects (font (size 12.7 12.7)) (justify left bottom))
   )
   (text "Debug/Log Header" (at 233.68 99.06 0)
@@
   )
   (text "WARNING: VBUS Backflow Possible\nWARNING: Significantly out of spec for power dissapation on MD5112\nWARNING: R10/R8 ARE INCORRECT FIX."
-    (at 1.27 124.46 0)
+    (at 2.54 125.73 0)
     (effects (font (size 1.27 1.27)) (justify left bottom))
   )
@@
       (effects (font (size 1.27 1.27)) (justify left))
     )
-    (property "Value" "10uH" (id 1) (at 251.46 41.91 0)
+    (property "Value" "4.7uH" (id 1) (at 251.46 41.91 0)
       (effects (font (size 1.27 1.27)) (justify left))
     )
@@
       (effects (font (size 1.27 1.27)) hide)
     )
-    (property "LCSC" "C356837" (id 4) (at 257.81 39.37 0)
+    (property "LCSC" "C379996" (id 4) (at 257.81 39.37 0)
       (effects (font (size 1.27 1.27)) hide)
     )
@@
   (symbol (lib_id "power:GND") (at 233.68 69.85 270) (unit 1)
     (in_bom yes) (on_board yes)
-    (property "Reference" "#PWR?" (id 0) (at 227.33 69.85 0)
+    (property "Reference" "#PWR0149" (id 0) (at 227.33 69.85 0)
       (effects (font (size 1.27 1.27)) hide)
     )
@@
     (in_bom yes) (on_board yes) (fields_autoplaced)
     (property "Reference" "L1" (id 0) (at 240.03 28.8122 90))
-    (property "Value" "10uH" (id 1) (at 240.03 31.3491 90))
+    (property "Value" "4.7uH" (id 1) (at 240.03 31.3491 90))
     (property "Footprint" "Inductor_SMD:L_0805_2012Metric" (id 2) (at 240.03 33.02 0)
       (effects (font (size 1.27 1.27)) hide)
@@
       (effects (font (size 1.27 1.27)) hide)
     )
-    (property "LCSC" "C356837" (id 4) (at 240.03 33.02 0)
+    (property "LCSC" "C379996" (id 4) (at 240.03 33.02 0)
       (effects (font (size 1.27 1.27)) hide)
     )
@@
       (reference "#PWR0148") (unit 1) (value "VDD") (footprint "")
     )
+    (path "/b9f5119b-f265-4871-ba2a-83a4810575e4"
+      (reference "#PWR0149") (unit 1) (value "GND") (footprint "")
+    )
     (path "/ff7c4d13-8004-4728-90b1-bcab92a74935"
       (reference "#PWR0150") (unit 1) (value "VD") (footprint "")
@@
       (reference "#PWR0162") (unit 1) (value "GND") (footprint "")
     )
-    (path "/b9f5119b-f265-4871-ba2a-83a4810575e4"
-      (reference "#PWR?") (unit 1) (value "GND") (footprint "")
-    )
     (path "/e2bd1966-aea5-4f9e-a70f-51c5a9f554dd"
       (reference "C1") (unit 1) (value "10u") (footprint "Capacitor_SMD:C_0402_1005Metric")
@@
     )
     (path "/c50ad1ea-c9dd-49db-93ef-f0a5c2aeda9e"
-      (reference "L1") (unit 1) (value "10uH") (footprint "Inductor_SMD:L_0805_2012Metric")
+      (reference "L1") (unit 1) (value "4.7uH") (footprint "Inductor_SMD:L_0805_2012Metric")
     )
     (path "/97803ad7-352c-4085-8487-f7735182611c"
-      (reference "L2") (unit 1) (value "10uH") (footprint "Inductor_SMD:L_0805_2012Metric")
+      (reference "L2") (unit 1) (value "4.7uH") (footprint "Inductor_SMD:L_0805_2012Metric")
     )
     (path "/13634884-96de-41e3-a90d-86653744f7db"

Commit message: Update design a little
Parts:
- Q2: footprint Package_TO_SOT_SMD:SOT-323_SC-70 -> DFN-3L-1x0.6:DFN-3L-1x0.6; LCSC C719079 -> C2875806
Other:
- note added: "FET Selection: * C2875806 -> ~250mO, 48pF * Inductors DCR: 110mO"
- moved on the sheet: C13, C15, D3, L1, L2, Q2, R16, R17
