File: hardware/ch32v003f4u6_pendant/VCCPSUSIM/VCCPSUSIM.kicad_sch (KiCad schematic)
At the start: 11 parts, among them Q1 Q_NMOS_DGS

Commit message: Switch over to using a .c file instead of a .S file for the startup code.  Helps make order-of-compiling not matter.
Parts:
- C1: Spice_Model 1u -> 12u
- C2: value 4.7uF -> cap; Spice_Model 1uF -> 1u
- L1: Spice_Model 4.7u -> 2.2u
- L2: Spice_Model 4.7uH -> 2.2u
- V2: Spice_Model pulse(0 3 2n 2n 2n 300n 500n) -> pulse(0 3 2n 2n 2n 100n 500n)
Changed lines of the file:
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@@
       (effects (font (size 1.27 1.27)) hide)
     )
-    (property "Spice_Model" "4.7uH" (id 5) (at 129.54 72.39 0))
+    (property "Spice_Model" "2.2u" (id 5) (at 129.54 72.39 0))
     (property "Spice_Netlist_Enabled" "Y" (id 6) (at 128.27 72.39 0)
       (effects (font (size 1.27 1.27)) hide)
@@
       (effects (font (size 1.27 1.27)) hide)
     )
-    (property "Spice_Model" "1u" (id 5) (at 116.84 48.26 0))
+    (property "Spice_Model" "12u" (id 5) (at 116.84 48.26 0))
     (property "Spice_Netlist_Enabled" "Y" (id 6) (at 116.84 48.26 0)
       (effects (font (size 1.27 1.27)) hide)
@@
       (effects (font (size 1.27 1.27)) (justify left) hide)
     )
-    (property "Spice_Model" "pulse(0 3 2n 2n 2n 300n 500n)" (id 6) (at 90.932 81.5209 0)
+    (property "Spice_Model" "pulse(0 3 2n 2n 2n 100n 500n)" (id 6) (at 90.932 81.5209 0)
       (effects (font (size 1.27 1.27)) (justify left))
     )
@@
       (effects (font (size 1.27 1.27)) hide)
     )
-    (property "Spice_Model" "4.7u" (id 5) (at 82.55 49.53 0))
+    (property "Spice_Model" "2.2u" (id 5) (at 82.55 49.53 0))
     (property "Spice_Netlist_Enabled" "Y" (id 6) (at 82.55 48.26 0)
       (effects (font (size 1.27 1.27)) hide)
@@
       (effects (font (size 1.27 1.27)) (justify right))
     )
-    (property "Value" "4.7uF" (id 1) (at 147.5541 59.69 90)
+    (property "Value" "cap" (id 1) (at 147.5541 59.69 90)
       (effects (font (size 1.27 1.27)) hide)
     )
@@
       (effects (font (size 1.27 1.27)) hide)
     )
-    (property "Spice_Model" "1uF" (id 5) (at 156.845 61.3922 0)
+    (property "Spice_Model" "1u" (id 5) (at 156.845 61.3922 0)
       (effects (font (size 1.27 1.27)) (justify right))
     )
@@
     )
     (path "/c53a62da-477d-4c9a-a34d-a0fa56d8902c"
-      (reference "C2") (unit 1) (value "4.7uF") (footprint "")
+      (reference "C2") (unit 1) (value "cap") (footprint "")
     )
     (path "/05e758ff-ca03-4ea4-a2f3-cb222ae8fc63"
