File: attic/hardware/ch32v003f4u6_pendant/ch32v003f4u6_pendant.kicad_pcb (KiCad board)
At the start: 2 copper layers, 20.3 x 51.4 mm, 52 parts, among them J1 USB_C_Receptacle_USB2.0, J2 BONUS, J3 BONUS, J4 CONN, J7 BATT, Q1 Q_Photo_NPN, Q2 NMOS, T1 TOUCHPAD, U1 MD5112, U2 CH32V003F4U6, U3 MD5112, U4 QMA7981, U5 RY2200, U6 RS3236-3.3YUTDN4, U7 S08OB383-031

Commit message: Update hardware
Parts:
- removed U1: MD5112, xdfn_reg:xdfn-reg
- added Q3: PNP, DFN-3L-1x0.6:DFN-3L-1x0.6, F.Cu at (101.5, 38.0)
- R6: value 15 -> 10k; footprint Resistor_SMD:R_0603_1608Metric -> Resistor_SMD:R_0402_1005Metric
- moved R9 10.5 mm to (92.5, 58.2), turned to -90 degrees
- moved R6 2.81 mm to (103.0, 36.2), turned to -90 degrees
- moved C3 0.46 mm to (104.9, 37.1)
Connections:
- R6 pad 1: Net-(C3-Pad1) -> GND
- R9 pad 1: NRST -> PA1
Routing:
- net VDD: track 59.6 -> 65.2 mm, vias 5 -> 7
- net Net-(C3-Pad1): track 5.90 -> 4.26 mm
- net NRST: track 13.0 -> 11.9 mm
- net Net-(C1-Pad1): track 11.4 -> 10.6 mm
- net GND: track 156.9 -> 157.7 mm
- net VD: track 70.5 -> 69.8 mm
