File: attic/hardware/ch32v003f4u6_pendant/ch32v003f4u6_pendant.kicad_sch (KiCad schematic)
At the start: 52 parts, among them J1 USB_C_Receptacle_USB2.0, J2 BONUS, J3 BONUS, J4 CONN, J7 BATT, Q1 Q_Photo_NPN, Q2 NMOS, T1 TOUCHPAD, U1 MD5112, U2 CH32V003F4U6, U3 MD5112, U4 QMA7981, U5 RY2200, U6 RS3236-3.3YUTDN4, U7 S08OB383-031

Commit message: Update hardware
Parts:
- removed U1: MD5112, xdfn_reg:xdfn-reg, symbol Regulator_Linear:NCP115AMX250TCG
- added Q3: PNP, DFN-3L-1x0.6:DFN-3L-1x0.6, symbol Device:Q_PNP_EBC
- C1: value 10u -> 2.2u; LCSC C315248 -> C385032
- R6: value 15 -> 10k; footprint Resistor_SMD:R_0603_1608Metric -> Resistor_SMD:R_0402_1005Metric; LCSC C402890 -> C269674
- U5: LCSC RY2200 -> C2888102
Connections:
- net GND: now also R6.1
- net NRST: no longer R9.1
- net PA1: now also R9.1
- net at C3.1, U3.3 (EN), U3.4 (IN): now also Q3.3 (C); no longer R6.1
- net at C1.1, J1.A4 (VBUS), J1.A9 (VBUS)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: now also Q3.1 (E)
- net at R6.2: now also Q3.2 (B)
Other:
- note added: "Note 1: VMON and Microphone are multiplexed VMON=1.06v nom at VCC=7v Mic is on highpass filter. Note 2: LM5112 V = 1.2v Note 2a: VDD is I and V limited. Note 2b: Ib is 0.5mA, Ic = ~60mA Note 2c: Charge Cutoff set to 4.1v Note 3: TBD: Can CH32 Pull-Down and ADC? Note 4: Jumper to test VDDMON Note 5: VCC Is a SEPIC Note 6: Is it possible to abuse NRST to measure voltage? Note 7: What should R8/R10 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"
- note added: "WARNING: VBUS Backflow Possible WARNING: R10/R8 ARE INCORRECT FIX."
- note removed: "Note 1: VMON and Microphone are multiplexed VMON=1.06v nom at VCC=7v Mic is on highpass filter. Note 2: LM5112 V = 1.2v Note 2a: VDD is I and V limited. Note 2b: Charge Current set to 80mA Note 2c: Charge Cutoff set to 4.1v Note 3: TBD: Can CH32 Pull-Down and ADC? Note 4: Jumper to test VDDMON Note 5: VCC Is a SEPIC Note 6: Is it possible to abuse NRST to measure voltage? Note 7: Do these MD5112'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"
- note removed: "Note 2b"
- note removed: "WARNING: VBUS Backflow Possible WARNING: Significantly out of spec for power dissapation on MD5112 WARNING: R10/R8 ARE INCORRECT FIX."
- moved on the sheet: R9
