File: attic/hardware/ch32v003f4u6_with_wsled_nomic/ch32v003f4u6_with_wsled.kicad_pcb (KiCad board)
At the start: 2 copper layers, 40.6 x 44.5 mm, 23 parts, among them J2 PGM, J4 USB_C_Receptacle_USB2.0, J5 HOLE, J6 HOLE, U1 CH32V003F4U6, U2 3.3vReg

Commit message: Update hardware
Parts:
- moved J4 0.10 mm to (100.0, 78.5)
Routing:
- net VCC: track 74.4 -> 70.7 mm, vias 11 -> 9
- net GND: vias 87 -> 89

Commit message: Update design and remove pendant.
Parts:
- added D7: LED, LED_SMD:LED_0402_1005Metric, F.Cu at (94.6, 84.9)
- added R6: 1.5k, Resistor_SMD:R_0402_1005Metric, F.Cu at (90.5, 101.7)
Routing:
- net Net-(D7-Pad2): track 0.00 -> 17.7 mm, vias 0 -> 2
- net GND: track 149.1 -> 145.2 mm, vias 89 -> 96
Other:
- board text added: "{dblquote}PC0{dblquote}"
