File: attic/hardware/ch32v003f4u6_with_wsled_nomic/ch32v003f4u6_with_wsled.kicad_sch (KiCad schematic)
At the start: 23 parts, among them J2 PGM, J4 USB_C_Receptacle_USB2.0, J5 HOLE, J6 HOLE, U1 CH32V003F4U6, U2 3.3vReg

Commit message: Update hardware
Parts:
- J1, J3: LCSC (none) -> C124359
- J2: LCSC C492404 -> C225257
Changed lines of the file:
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@@
       (effects (font (size 1.27 1.27)) hide)
     )
-    (property "LCSC" "C492404" (id 4) (at 96.52 143.51 0)
+    (property "LCSC" "C225257" (id 4) (at 96.52 143.51 0)
       (effects (font (size 1.27 1.27)) hide)
     )
@@
     )
     (property "Datasheet" "~" (id 3) (at 35.56 104.14 0)
+      (effects (font (size 1.27 1.27)) hide)
+    )
+    (property "LCSC" "C124359" (id 4) (at 35.56 104.14 0)
       (effects (font (size 1.27 1.27)) hide)
     )
@@
       (effects (font (size 1.27 1.27)) hide)
     )
+    (property "LCSC" "C124359" (id 4) (at 193.04 104.14 0)
+      (effects (font (size 1.27 1.27)) hide)
+    )

Commit message: Update design and remove pendant.
Parts:
- added D7: LED, LED_SMD:LED_0402_1005Metric, symbol Device:LED
- added R6: 1.5k, Resistor_SMD:R_0402_1005Metric, symbol Device:R
Connections:
- net GND: now also D7.1 (K)
- net PC0: now also R6.2
- new net: D7.2 (A), R6.1
Changed lines of the file:
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@@
+    )
+  )
+  (global_label "PC0" (shape input) (at 199.39 134.62 180) (fields_autoplaced)
+    (effects (font (size 1.27 1.27)) (justify right))
+    (property "Intersheet References" "${INTERSHEET_REFS}" (id 0) (at 193.2274 134.5406 0)
+      (effects (font (size 1.27 1.27)) (justify right) hide)
     )
   )
@@
     (pin "1")
   )
+  (symbol (lib_id "Device:R") (at 199.39 138.43 180) (unit 1)
+    (in_bom yes) (on_board yes)
+    (property "Reference" "R6" (id 0) (at 203.2 137.16 0))
+    (property "Value" "1.5k" (id 1) (at 203.2 139.7 0))
+    (property "Footprint" "Resistor_SMD:R_0402_1005Metric" (id 2) (at 201.168 138.43 90)
+      (effects (font (size 1.27 1.27)) hide)
+    )
+    (property "Datasheet" "~" (id 3) (at 199.39 138.43 0)
+      (effects (font (size 1.27 1.27)) hide)
+    )
+    (property "LCSC" "C25867" (id 4) (at 199.39 138.43 90)
+      (effects (font (size 1.27 1.27)) hide)
+    )
+    (pin "1")
+    (pin "2")
+  )
   (symbol (lib_id "power:VD") (at 179.07 60.96 90) (unit 1)
     (in_bom yes) (on_board yes) (fields_autoplaced)
@@
     )
     (pin "1")
+  )
+  (symbol (lib_id "Device:LED") (at 199.39 146.05 90) (unit 1)
+    (in_bom yes) (on_board yes)
+    (property "Reference" "D7" (id 0) (at 203.2 144.78 90))
+    (property "Value" "LED" (id 1) (at 203.2 147.32 90))
+    (property "Footprint" "LED_SMD:LED_0402_1005Metric" (id 2) (at 199.39 146.05 0)
+      (effects (font (size 1.27 1.27)) hide)
+    )
+    (property "Datasheet" "~" (id 3) (at 199.39 146.05 0)
+      (effects (font (size 1.27 1.27)) hide)
+    )
+    (property "LCSC" "C74342" (id 4) (at 199.39 146.05 0)
+      (effects (font (size 1.27 1.27)) hide)
+    )
+    (pin "1")
+    (pin "2")
   )
   (symbol (lib_id "power:GND") (at 119.38 58.42 0) (unit 1)
@@
     )
     (property "Datasheet" "" (id 3) (at 43.18 106.68 0)
+      (effects (font (size 1.27 1.27)) hide)
+    )
+    (pin "1")
+  )
+  (symbol (lib_id "power:GND") (at 199.39 149.86 0) (unit 1)
+    (in_bom yes) (on_board yes) (fields_autoplaced)
+    (property "Reference" "#PWR01" (id 0) (at 199.39 156.21 0)
+      (effects (font (size 1.27 1.27)) hide)
+    )
+    (property "Value" "GND" (id 1) (at 199.39 154.94 0))
+    (property "Footprint" "" (id 2) (at 199.39 149.86 0)
+      (effects (font (size 1.27 1.27)) hide)
+    )
+    (property "Datasheet" "" (id 3) (at 199.39 149.86 0)
       (effects (font (size 1.27 1.27)) hide)
     )
@@
   )
   (symbol_instances
+    (path "/b6d95e52-9c0e-4cbc-819a-6c2785b5bd34"
+      (reference "#PWR01") (unit 1) (value "GND") (footprint "")
+    )
     (path "/5399c7c8-9c50-4f58-94d1-5ef1a660ca5c"
       (reference "#PWR09") (unit 1) (value "GND") (footprint "")
@@
       (reference "D6") (unit 1) (value "WS2816C-2121") (footprint "WS2816-2121:WS2816-2121")
     )
+    (path "/a325821d-8a54-4a3b-981a-ca0742a104c5"
+      (reference "D7") (unit 1) (value "LED") (footprint "LED_SMD:LED_0402_1005Metric")
+    )
     (path "/7b320334-9555-4edf-874c-a98a073a480a"
       (reference "J1") (unit 1) (value "~") (footprint "Connector_PinHeader_2.54mm:PinHeader_2x10_P2.54mm_Vertical")
@@
       (reference "R5") (unit 1) (value "NP") (footprint "Resistor_SMD:R_0402_1005Metric")
     )
+    (path "/9ff23070-8d50-4c43-9132-802478518421"
+      (reference "R6") (unit 1) (value "1.5k") (footprint "Resistor_SMD:R_0402_1005Metric")
+    )
     (path "/8e4967a9-bbc0-4179-bc6b-41548631bd33"
